File: schematic/MCBUPS/sheet1.kicad_sch (KiCad schematic)
At the start: 47 parts, among them Q2 BC547, U1 LM324, U2 4098

Commit message: MCBUPS board was working
Parts:
- C10, C4, C6: value C -> 100nF
- C5, C8: value C_P -> 100uF
- C7: value C_P -> 22uF
- R10: value R -> 10k
- R96: value 560k -> 100k
- RV5: value 5k -> 100k
Changed lines of the file:
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@@
 			)
 		)
-		(property "Value" "560k"
+		(property "Value" "100k"
 			(at 75.565 31.115 90)
 			(effects
@@
 			)
 		)
-		(property "Value" "C"
+		(property "Value" "100nF"
 			(at 186.055 97.79 90)
 			(effects
@@
 		(fields_autoplaced yes)
 		(property "Reference" "R10"
-			(at 20.955 80.6449 0)
+			(at 20.32 80.6449 0)
 			(effects
 				(font
@@
 			)
 		)
-		(property "Value" "R"
-			(at 20.955 83.1849 0)
+		(property "Value" "10k"
+			(at 20.32 83.1849 0)
 			(effects
 				(font
@@
 			)
 		)
-		(property "Value" "C"
+		(property "Value" "100nF"
 			(at 223.52 114.3 90)
 			(effects
@@
 		(fields_autoplaced yes)
 		(property "Reference" "C5"
-			(at 235.585 150.8759 0)
+			(at 236.22 150.8759 0)
 			(effects
 				(font
@@
 			)
 		)
-		(property "Value" "C_P"
-			(at 235.585 153.4159 0)
+		(property "Value" "100uF"
+			(at 236.22 153.4159 0)
 			(effects
 				(font
@@
 			)
 		)
-		(property "Value" "C_P"
+		(property "Value" "22uF"
 			(at 190.881 82.55 90)
 			(effects
@@
 			)
 		)
-		(property "Value" "C"
+		(property "Value" "100nF"
 			(at 27.94 137.7949 0)
 			(effects
@@
 			)
 		)
-		(property "Value" "5k"
+		(property "Value" "100k"
 			(at 74.295 50.1651 90)
 			(effects
@@
 			)
 		)
-		(property "Value" "C_P"
+		(property "Value" "100uF"
 			(at 36.83 44.8309 0)
 			(effects
