File: schematic/MCBUPS/sheet3.kicad_sch (KiCad schematic)
At the start: 53 parts, among them Q1 BC547, Q10 BC547, Q11 BC557, Q12 BC547, Q15 BC557, Q20 BC547, U4 SG3524N

Commit message: MCBUPS board was working
Parts:
- C1, C9: value C -> 100nF
- C11, C25: value C_P -> 10uF
- C23: value C_P -> 1uF
- R47: value R -> 4.7k
Changed lines of the file:
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@@
 			)
 		)
-		(property "Value" "C_P"
+		(property "Value" "10uF"
 			(at 121.92 107.6959 0)
 			(effects
@@
 			)
 		)
-		(property "Value" "R"
+		(property "Value" "4.7k"
 			(at 160.655 24.13 90)
 			(effects
@@
 		(fields_autoplaced yes)
 		(property "Reference" "C1"
-			(at 136.525 105.4099 0)
+			(at 135.89 105.4099 0)
 			(effects
 				(font
@@
 			)
 		)
-		(property "Value" "C"
-			(at 136.525 107.9499 0)
+		(property "Value" "100nF"
+			(at 135.89 107.9499 0)
 			(effects
 				(font
@@
 			)
 		)
-		(property "Value" "C"
+		(property "Value" "100nF"
 			(at 173.99 88.265 0)
 			(effects
@@
 		(fields_autoplaced yes)
 		(property "Reference" "C11"
-			(at 136.525 35.3059 0)
+			(at 135.89 35.3059 0)
 			(effects
 				(font
@@
 			)
 		)
-		(property "Value" "C_P"
-			(at 136.525 37.8459 0)
+		(property "Value" "10uF"
+			(at 135.89 37.8459 0)
 			(effects
 				(font
@@
 			)
 		)
-		(property "Value" "C_P"
+		(property "Value" "1uF"
 			(at 158.75 87.3759 0)
 			(effects
