File: schematic/MCBUPS/sheet4.kicad_sch (KiCad schematic)
At the start: 38 parts, among them Q5 SL100, Q6 SL100, Q7 SL100, U3 LM324

Commit message: MCBUPS board was working
Parts:
- added R112: 2.2k, symbol PCM_Elektuur:R
- C13: value C_P -> 47uF
- C14: value C_P -> 10uF
- R30, R33, R38, R43: value R -> 100k
- R39, R42: value R -> 1k
- R41: value R -> 2.2k
- R77: value 2.2k -> 1k
- R82: value 5.7k -> 2.7k
- RV7: value 5k -> 20k
- RV8: value 5k -> 10k
Connections:
- net GND: now also R112.1 (+)
- net at C14.1, R39.1 (+), R78.1 (+)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: now also R112.2 (-)
Changed lines of the file:
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@@
 	)
 	(junction
+		(at 68.58 170.18)
+		(diameter 0)
+		(color 0 0 0 0)
+	)
+	(junction
 		(at 139.065 49.53)
 		(diameter 0)
@@
 	(wire
 		(pts
+			(xy 68.58 182.245) (xy 68.58 184.15)
+		)
+		(stroke
+			(width 0)
+			(type default)
+		)
+	)
+	(wire
+		(pts
 			(xy 38.1 49.53) (xy 38.1 52.07)
 		)
@@
 		)
 	)
+	(wire
+		(pts
+			(xy 68.58 170.18) (xy 68.58 172.085)
+		)
+		(stroke
+			(width 0)
+			(type default)
+		)
+	)
 	(label "J2_RL0"
 		(at 163.83 41.91 180)
@@
 			)
 		)
-		(property "Value" "5k"
+		(property "Value" "20k"
 			(at 76.835 65.4051 90)
 			(effects
@@
 			)
 		)
-		(property "Value" "R"
+		(property "Value" "2.2k"
 			(at 81.28 135.8899 0)
 			(effects
@@
 			)
 		)
-		(property "Value" "R"
+		(property "Value" "100k"
 			(at 106.045 139.065 90)
 			(effects
@@
 			)
 		)
-		(property "Value" "R"
+		(property "Value" "100k"
 			(at 107.315 115.57 90)
 			(effects
@@
 		(fields_autoplaced yes)
 		(property "Reference" "C13"
-			(at 41.275 43.5609 0)
+			(at 41.91 43.5609 0)
 			(effects
 				(font
@@
 			)
 		)
-		(property "Value" "C_P"
-			(at 41.275 46.1009 0)
+		(property "Value" "47uF"
+			(at 41.91 46.1009 0)
 			(effects
 				(font
@@
 	)
 	(symbol
+		(lib_id "PCM_Elektuur:R")
+		(at 68.58 177.165 180)
+		(unit 1)
+		(exclude_from_sim no)
+		(in_bom yes)
+		(on_board yes)
+		(dnp no)
+		(property "Reference" "R112"
+			(at 71.755 175.8949 0)
+			(effects
+				(font
+					(size 1.27 1.27)
+				)
+				(justify right)
+			)
+		)
+		(property "Value" "2.2k"
+			(at 71.755 178.4349 0)
+			(effects
+				(font
+					(size 1.27 1.27)
+				)
+				(justify right)
+			)
+		)
+		(property "Footprint" ""
+			(at 68.58 177.165 0)
+			(effects
+				(font
+					(size 1.27 1.27)
+				)
+				(hide yes)
+			)
+		)
+		(property "Datasheet" ""
+			(at 68.58 177.165 0)
+			(effects
+				(font
+					(size 1.27 1.27)
+				)
+				(hide yes)
+			)
+		)
+		(property "Description" "resistor"
+			(at 68.58 177.165 0)
+			(effects
+				(font
+					(size 1.27 1.27)
+				)
+				(hide yes)
+			)
+		)
+		(property "Indicator" "+"
+			(at 71.755 180.34 0)
+			(effects
+				(font
+					(size 1.27 1.27)
+				)
+				(hide yes)
+			)
+		)
+		(property "Rating" "W"
+			(at 66.04 173.99 0)
+			(effects
+				(font
+					(size 1.27 1.27)
+				)
+				(justify left)
+				(hide yes)
+			)
+		)
+		(pin "2"
+		)
+		(pin "1"
+		)
+		(instances
+			(project "MCBUPS"
+				(path "/bce3dcac-4a87-4902-86a6-a59da237e6a9/5f428e04-1417-41b3-90f8-d762af1aaa33"
+					(reference "R112")
+					(unit 1)
+				)
+			)
+		)
+	)
+	(symbol
 		(lib_id "power:+8V")
 		(at 78.74 48.895 0)
@@
 			)
 		)
-		(property "Value" "5k"
+		(property "Value" "10k"
 			(at 76.835 101.6001 90)
 			(effects
@@
 			)
 		)
-		(property "Value" "R"
+		(property "Value" "1k"
 			(at 88.265 167.64 90)
 			(effects
@@
 	)
 	(symbol
+		(lib_id "power:GND")
+		(at 68.58 184.15 0)
+		(unit 1)
+		(exclude_from_sim no)
+		(in_bom yes)
+		(on_board yes)
+		(dnp no)
+		(fields_autoplaced yes)
+		(property "Reference" "#PWR02"
+			(at 68.58 190.5 0)
+			(effects
+				(font
+					(size 1.27 1.27)
+				)
+				(hide yes)
+			)
+		)
+		(property "Value" "GND"
+			(at 68.58 188.595 0)
+			(effects
+				(font
+					(size 1.27 1.27)
+				)
+			)
+		)
+		(property "Footprint" ""
+			(at 68.58 184.15 0)
+			(effects
+				(font
+					(size 1.27 1.27)
+				)
+				(hide yes)
+			)
+		)
+		(property "Datasheet" ""
+			(at 68.58 184.15 0)
+			(effects
+				(font
+					(size 1.27 1.27)
+				)
+				(hide yes)
+			)
+		)
+		(property "Description" "Power symbol creates a global label with name \"GND\" , ground"
+			(at 68.58 184.15 0)
+			(effects
+				(font
+					(size 1.27 1.27)
+				)
+				(hide yes)
+			)
+		)
+		(pin "1"
+		)
+		(instances
+			(project "MCBUPS"
+				(path "/bce3dcac-4a87-4902-86a6-a59da237e6a9/5f428e04-1417-41b3-90f8-d762af1aaa33"
+					(reference "#PWR02")
+					(unit 1)
+				)
+			)
+		)
+	)
+	(symbol
 		(lib_id "PCM_Elektuur:R")
 		(at 86.995 143.51 90)
@@
 			)
 		)
-		(property "Value" "R"
+		(property "Value" "1k"
 			(at 86.995 139.065 90)
 			(effects
@@
 			)
 		)
-		(property "Value" "R"
+		(property "Value" "100k"
 			(at 107.315 167.64 90)
 			(effects
@@
 		(fields_autoplaced yes)
 		(property "Reference" "C14"
-			(at 64.135 44.1959 0)
+			(at 64.77 44.1959 0)
 			(effects
 				(font
@@
 			)
 		)
-		(property "Value" "C_P"
-			(at 64.135 46.7359 0)
+		(property "Value" "10uF"
+			(at 64.77 46.7359 0)
 			(effects
 				(font
@@
 		(fields_autoplaced yes)
 		(property "Reference" "R82"
-			(at 81.915 90.1699 0)
+			(at 81.28 90.1699 0)
 			(effects
 				(font
@@
 			)
 		)
-		(property "Value" "5.7k"
-			(at 81.915 92.7099 0)
+		(property "Value" "2.7k"
+			(at 81.28 92.7099 0)
 			(effects
 				(font
@@
 		(fields_autoplaced yes)
 		(property "Reference" "R77"
-			(at 81.915 53.9749 0)
+			(at 81.28 53.9749 0)
 			(effects
 				(font
@@
 			)
 		)
-		(property "Value" "2.2k"
-			(at 81.915 56.5149 0)
+		(property "Value" "1k"
+			(at 81.28 56.5149 0)
 			(effects
 				(font
@@
 			)
 		)
-		(property "Value" "R"
+		(property "Value" "100k"
 			(at 107.315 57.15 90)
 			(effects
