File: schematic/MCBUPS/untitled.kicad_sch (KiCad schematic)
At the start: 65 parts, among them Q0 SL100, Q13 BC547, Q3 BC547, Q4 SL100, U5 LM324, U6 LM324

Commit message: MCBUPS board was working
Parts:
- removed C16: C_P, symbol Device:C_Polarized
- added R29: 1k, symbol PCM_Elektuur:R
- C17: value C_P -> 100uF
- C18, C19: value C_P -> 4.7uF
- R111: value R -> 2.2k
- R18: value 1.5k -> 15k
- R5: value 2.2k -> 4.7k
- R60: value R -> 100
- R61: value 820k -> 8.2k
- R62: value R -> 12k
- R64: value R -> 47k
- R70: value R -> 10k
- R86: value R -> 470ohm
- R88: value R -> 1k
- RV1: value 5k -> 100k
- RV4: value 5k -> 10k
Connections:
- net GND: now also R29.2 (-)
- net at R65.1 (+), RV4.2, RV4.3: now also R29.1 (+)
Changed lines of the file:
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@@
 	(wire
 		(pts
-			(xy 183.515 41.275) (xy 183.515 138.43)
+			(xy 259.715 46.99) (xy 259.715 48.895)
 		)
 		(stroke
@@
 	(wire
 		(pts
-			(xy 120.65 160.655) (xy 120.65 163.83)
+			(xy 183.515 41.275) (xy 183.515 138.43)
 		)
 		(stroke
@@
 	(wire
 		(pts
-			(xy 104.14 93.345) (xy 96.52 93.345)
+			(xy 120.65 160.655) (xy 120.65 163.83)
 		)
 		(stroke
@@
 	(wire
 		(pts
-			(xy 252.095 70.485) (xy 255.905 70.485)
+			(xy 104.14 93.345) (xy 96.52 93.345)
 		)
 		(stroke
@@
 	(wire
 		(pts
-			(xy 259.715 44.45) (xy 259.715 47.625)
+			(xy 252.095 70.485) (xy 255.905 70.485)
 		)
 		(stroke
@@
 			)
 		)
-		(property "Value" "5k"
+		(property "Value" "10k"
 			(at 261.62 25.4001 90)
 			(effects
@@
 			)
 		)
-		(property "Value" "5k"
+		(property "Value" "100k"
 			(at 135.89 179.7051 90)
 			(effects
@@
 	)
 	(symbol
+		(lib_id "PCM_Elektuur:R")
+		(at 259.715 41.91 0)
+		(unit 1)
+		(exclude_from_sim no)
+		(in_bom yes)
+		(on_board yes)
+		(dnp no)
+		(property "Reference" "R29"
+			(at 266.7 41.91 90)
+			(effects
+				(font
+					(size 1.27 1.27)
+				)
+			)
+		)
+		(property "Value" "1k"
+			(at 264.16 41.91 90)
+			(effects
+				(font
+					(size 1.27 1.27)
+				)
+			)
+		)
+		(property "Footprint" ""
+			(at 259.715 41.91 0)
+			(effects
+				(font
+					(size 1.27 1.27)
+				)
+				(hide yes)
+			)
+		)
+		(property "Datasheet" ""
+			(at 259.715 41.91 0)
+			(effects
+				(font
+					(size 1.27 1.27)
+				)
+				(hide yes)
+			)
+		)
+		(property "Description" "resistor"
+			(at 259.715 41.91 0)
+			(effects
+				(font
+					(size 1.27 1.27)
+				)
+				(hide yes)
+			)
+		)
+		(property "Indicator" "+"
+			(at 256.54 38.735 0)
+			(effects
+				(font
+					(size 1.27 1.27)
+				)
+				(hide yes)
+			)
+		)
+		(property "Rating" "W"
+			(at 262.255 45.085 0)
+			(effects
+				(font
+					(size 1.27 1.27)
+				)
+				(justify left)
+				(hide yes)
+			)
+		)
+		(pin "2"
+		)
+		(pin "1"
+		)
+		(instances
+			(project "MCBUPS"
+				(path "/bce3dcac-4a87-4902-86a6-a59da237e6a9/1700017d-79a5-4253-a71a-2b4cabddbef2"
+					(reference "R29")
+					(unit 1)
+				)
+			)
+		)
+	)
+	(symbol
 		(lib_id "Simulation_SPICE:NPN")
 		(at 88.265 118.745 0)
@@
 			)
 		)
-		(property "Value" "R"
+		(property "Value" "1k"
 			(at 54.61 163.1949 0)
 			(effects
@@
 		(fields_autoplaced yes)
 		(property "Reference" "R18"
-			(at 267.335 91.4399 0)
+			(at 266.7 91.4399 0)
 			(effects
 				(font
@@
 			)
 		)
-		(property "Value" "1.5k"
-			(at 267.335 93.9799 0)
+		(property "Value" "15k"
+			(at 266.7 93.9799 0)
 			(effects
 				(font
@@
 			)
 		)
-		(property "Value" "C_P"
+		(property "Value" "100uF"
 			(at 43.815 162.56 0)
 			(effects
@@
 		(fields_autoplaced yes)
 		(property "Reference" "C27"
-			(at 160.655 48.6409 0)
+			(at 161.29 48.6409 0)
 			(effects
 				(font
@@
 		)
 		(property "Value" "C_P"
-			(at 160.655 51.1809 0)
+			(at 161.29 51.1809 0)
 			(effects
 				(font
@@
 			)
 		)
-		(property "Value" "C_P"
+		(property "Value" "4.7uF"
 			(at 116.84 158.115 0)
 			(effects
@@
 			)
 		)
-		(property "Value" "R"
+		(property "Value" "10k"
 			(at 77.47 134.62 90)
 			(effects
@@
 			)
 		)
-		(property "Value" "R"
+		(property "Value" "2.2k"
 			(at 203.835 130.175 90)
 			(effects
@@
 			)
 		)
-		(property "Value" "R"
+		(property "Value" "12k"
 			(at 247.015 66.04 90)
 			(effects
@@
 			)
 		)
-		(property "Value" "C_P"
+		(property "Value" "4.7uF"
 			(at 94.615 158.115 0)
 			(effects
@@
 			)
 		)
-		(property "Value" "820k"
+		(property "Value" "8.2k"
 			(at 251.46 131.445 90)
 			(effects
@@
 	)
 	(symbol
-		(lib_id "Device:C_Polarized")
-		(at 259.715 40.64 0)
-		(mirror y)
-		(unit 1)
-		(exclude_from_sim no)
-		(in_bom yes)
-		(on_board yes)
-		(dnp no)
-		(fields_autoplaced yes)
-		(property "Reference" "C16"
-			(at 255.905 38.4809 0)
-			(effects
-				(font
-					(size 1.27 1.27)
-				)
-				(justify left)
-			)
-		)
-		(property "Value" "C_P"
-			(at 255.905 41.0209 0)
-			(effects
-				(font
-					(size 1.27 1.27)
-				)
-				(justify left)
-			)
-		)
-		(property "Footprint" ""
-			(at 258.7498 44.45 0)
-			(effects
-				(font
-					(size 1.27 1.27)
-				)
-				(hide yes)
-			)
-		)
-		(property "Datasheet" "~"
-			(at 259.715 40.64 0)
-			(effects
-				(font
-					(size 1.27 1.27)
-				)
-				(hide yes)
-			)
-		)
-		(property "Description" "Polarized capacitor"
-			(at 259.715 40.64 0)
-			(effects
-				(font
-					(size 1.27 1.27)
-				)
-				(hide yes)
-			)
-		)
-		(pin "1"
-		)
-		(pin "2"
-		)
-		(instances
-			(project "MCBUPS"
-				(path "/bce3dcac-4a87-4902-86a6-a59da237e6a9/1700017d-79a5-4253-a71a-2b4cabddbef2"
-					(reference "C16")
-					(unit 1)
-				)
-			)
-		)
-	)
-	(symbol
 		(lib_id "PCM_Elektuur:R")
 		(at 67.945 99.695 90)
@@
 			)
 		)
-		(property "Value" "R"
+		(property "Value" "47k"
 			(at 245.745 92.075 90)
 			(effects
@@
 			)
 		)
-		(property "Value" "2.2k"
+		(property "Value" "4.7k"
 			(at 122.555 93.98 90)
 			(effects
@@
 			)
 		)
-		(property "Value" "R"
+		(property "Value" "100"
 			(at 234.315 88.9 90)
 			(effects
@@
 	(symbol
 		(lib_id "power:GND")
-		(at 259.715 47.625 0)
+		(at 259.715 48.895 0)
 		(mirror y)
 		(unit 1)
@@
 		(fields_autoplaced yes)
 		(property "Reference" "#PWR055"
-			(at 259.715 53.975 0)
+			(at 259.715 55.245 0)
 			(effects
 				(font
@@
 		)
 		(property "Value" "GND"
-			(at 259.715 52.07 0)
+			(at 259.715 53.34 0)
 			(effects
 				(font
@@
 		)
 		(property "Footprint" ""
-			(at 259.715 47.625 0)
+			(at 259.715 48.895 0)
 			(effects
 				(font
@@
 		)
 		(property "Datasheet" ""
-			(at 259.715 47.625 0)
+			(at 259.715 48.895 0)
 			(effects
 				(font
@@
 		)
 		(property "Description" "Power symbol creates a global label with name \"GND\" , ground"
-			(at 259.715 47.625 0)
+			(at 259.715 48.895 0)
 			(effects
 				(font
@@
 			)
 		)
-		(property "Value" "R"
+		(property "Value" "470ohm"
 			(at 105.41 158.7499 0)
 			(effects
